File: Windtunnel_Schematic/arduino_nano.kicad_sch (KiCad schematic)
At the start: 1 part

Commit message: Schematic to 0.3.0 Nearly finished Trying to mill it tomorrow
Connections:
- net D11: now also A1.13 (D10); no longer A1.14 (D11)
- net D12: now also A1.14 (D11); no longer A1.15 (D12)
- net D13: now also A1.15 (D12); no longer A1.16 (D13)
Changed lines of the file:
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@@
 	(title_block
 		(title "Schematic for wind tunnel measurement system")
-		(rev "0.2.0")
+		(rev "0.3.0")
 		(company "Reykjavik University")
 	)
@@
 	)
 	(no_connect
+		(at 146.05 96.52)
+	)
+	(no_connect
 		(at 156.21 53.34)
 	)
@@
 	)
 	(no_connect
-		(at 146.05 88.9)
-	)
-	(no_connect
 		(at 146.05 71.12)
 	)
@@
 	(wire
 		(pts
+			(xy 140.97 88.9) (xy 146.05 88.9)
+		)
+		(stroke
+			(width 0)
+			(type default)
+		)
+	)
+	(wire
+		(pts
 			(xy 140.97 81.28) (xy 146.05 81.28)
 		)
@@
 	(wire
 		(pts
-			(xy 140.97 96.52) (xy 146.05 96.52)
-		)
-		(stroke
-			(width 0)
-			(type default)
-		)
-	)
-	(wire
-		(pts
 			(xy 140.97 73.66) (xy 146.05 73.66)
 		)
@@
 	(wire
 		(pts
+			(xy 158.75 105.41) (xy 161.29 105.41)
+		)
+		(stroke
+			(width 0)
+			(type default)
+		)
+	)
+	(wire
+		(pts
+			(xy 171.45 88.9) (xy 182.88 88.9)
+		)
+		(stroke
+			(width 0)
+			(type default)
+		)
+	)
+	(wire
+		(pts
+			(xy 171.45 91.44) (xy 182.88 91.44)
+		)
+		(stroke
+			(width 0)
+			(type default)
+		)
+	)
+	(wire
+		(pts
 			(xy 140.97 91.44) (xy 146.05 91.44)
 		)
@@
 	(wire
 		(pts
-			(xy 158.75 105.41) (xy 161.29 105.41)
-		)
-		(stroke
-			(width 0)
-			(type default)
-		)
-	)
-	(wire
-		(pts
 			(xy 140.97 93.98) (xy 146.05 93.98)
-		)
-		(stroke
-			(width 0)
-			(type default)
-		)
-	)
-	(wire
-		(pts
-			(xy 171.45 88.9) (xy 182.88 88.9)
-		)
-		(stroke
-			(width 0)
-			(type default)
-		)
-	)
-	(wire
-		(pts
-			(xy 171.45 91.44) (xy 182.88 91.44)
 		)
 		(stroke
@@
 	(hierarchical_label "D12"
 		(shape bidirectional)
-		(at 140.97 93.98 180)
+		(at 140.97 91.44 180)
 		(fields_autoplaced yes)
 		(effects
@@
 	(hierarchical_label "D11"
 		(shape bidirectional)
-		(at 140.97 91.44 180)
+		(at 140.97 88.9 180)
 		(fields_autoplaced yes)
 		(effects
@@
 	(hierarchical_label "D13"
 		(shape bidirectional)
-		(at 140.97 96.52 180)
-		(fields_autoplaced yes)
-		(effects
+		(at 140.97 93.98 180)
+		(fields_autoplaced yes)
+		(effects

Commit message: Add to docs, schematic and general calculation: ADD prototype data Change Schematic revision to 0.4.0 ADD requirements.txt for each general calculation virtual environment
Connections:
- net D11 renamed D10_Rst_Tare
- net D12 renamed D11_Tare_Drag
- net D13 renamed D12_Tare_Lift
Changed lines of the file:
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@@
 	(title_block
 		(title "Schematic for wind tunnel measurement system")
-		(rev "0.3.0")
+		(rev "0.4.0")
 		(company "Reykjavik University")
 	)
@@
 		)
 	)
-	(hierarchical_label "D12"
+	(hierarchical_label "D11_Tare_Drag"
 		(shape bidirectional)
 		(at 140.97 91.44 180)
@@
 		)
 	)
-	(hierarchical_label "D11"
+	(hierarchical_label "D10_Rst_Tare"
 		(shape bidirectional)
 		(at 140.97 88.9 180)
@@
 		)
 	)
-	(hierarchical_label "D13"
+	(hierarchical_label "D12_Tare_Lift"
 		(shape bidirectional)
 		(at 140.97 93.98 180)
